File: Hardware/PCB-Mando-Radiocontrol/PCB-Mando-Radiocontrol/PCB-Mando-Radiocontrol-backups.kicad_pcb (KiCad board)
At the start: 2 copper layers, 132 x 66 mm, 25 parts, among them J1 nombre del prog, U1 ATMEGA328P, U2 Nrf24l01, U3 AMS1117-3.3, U4 AMS1117-5.0, U5 COM-09032, U6 COM-09032, Y1 16MHZ

Commit message: Avances en el PCB de la controladora de vuelo
Parts:
- J1: value nombre del prog -> USB 2.0 a UART TTL 6 pines CP2102
Connections:
- J1 pad 4: unconnected-(J1-Pin_4-Pad4) -> +5V
- J1 pad 5: unconnected-(J1-Pin_5-Pad5) -> GND
- J1 pad 6: GND -> unconnected-(J1-Pin_6-Pad6)
- U1 pad 20: GND -> +5V
- U1 pad 22: +5V -> GND
