File: Hardware/PCB-Controladora-Vuelo/PCB_Controladora_Vuelo_V2/PCB_Controladora_Vuelo_V2.kicad_pcb (KiCad board)
At the start: 2 copper layers, 40 x 92 mm, 14 parts, among them J1 Jumper Serial, J2 ESC, U1 MPU-5060, U2 ESP32-DEVKIT-V1, U3 Nrf24l01, U4 AMS1117-3.3

Commit message: Modificaciones finales en la V2 del PCB de la FC
Parts:
- C1, C5: footprint Capacitor_SMD:C_1206_3216Metric_Pad1.33x1.80mm_HandSolder -> EESTN5:C_0805
- C3, C7: footprint Capacitor_SMD:C_1206_3216Metric -> EESTN5:C_0805
- moved C5 3.08 mm to (116.3, 66.1), turned to 90 degrees
- moved C7 1.22 mm to (116.3, 61.1), turned to -90 degrees
- moved C1 1.18 mm to (130.2, 61.1), turned to 90 degrees
- moved C3 1.00 mm to (130.2, 66.1), turned to -90 degrees
Routing:
- net GND: track 32.3 -> 27.9 mm
- net +5V: track 83.1 -> 80.6 mm
- net +3V3: track 222.9 -> 222.4 mm
