File: Hardware/PCB-Controladora-Vuelo/PCB_Controladora_Vuelo_V2/PCB_Controladora_Vuelo_V2.kicad_sch (KiCad schematic)
At the start: 14 parts, among them J1 Jumper Serial, J2 ESC, U1 MPU-5060, U2 ESP32-DEVKIT-V1, U2 Nrf24l01, U3 AMS1117-3.3

Commit message: Modificaciones finales en la V2 del PCB de la FC
Parts:
- C5, C7: footprint Capacitor_SMD:C_1206_3216Metric_Pad1.33x1.80mm_HandSolder -> EESTN5:C_0805
- C6, C8: footprint Capacitor_SMD:C_1206_3216Metric -> EESTN5:C_0805
Changed lines of the file:
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@@
     (pin "1")
     (instances
-      (project "PCB-Controladora-Vuelo"
+      (project "PCB_Controladora_Vuelo_V2"
         (path "/ac5864b2-231c-45bd-8efa-594ea27cde2d"
           (reference "#PWR018") (unit 1)
@@
     (pin "S2")
     (instances
-      (project "PCB-Controladora-Vuelo"
+      (project "PCB_Controladora_Vuelo_V2"
         (path "/ac5864b2-231c-45bd-8efa-594ea27cde2d"
           (reference "J2") (unit 1)
@@
     )
     (instances
-      (project "PCB-Controladora-Vuelo"
+      (project "PCB_Controladora_Vuelo_V2"
         (path "/ac5864b2-231c-45bd-8efa-594ea27cde2d"
           (reference "H2") (unit 1)
@@
     )
     (instances
-      (project "PCB-Controladora-Vuelo"
+      (project "PCB_Controladora_Vuelo_V2"
         (path "/ac5864b2-231c-45bd-8efa-594ea27cde2d"
           (reference "H1") (unit 1)
@@
         )
       )
-      (project "PCB-Controladora-Vuelo"
+      (project "PCB_Controladora_Vuelo_V2"
         (path "/ac5864b2-231c-45bd-8efa-594ea27cde2d"
           (reference "#PWR06") (unit 1)
@@
         )
       )
-      (project "PCB-Controladora-Vuelo"
+      (project "PCB_Controladora_Vuelo_V2"
         (path "/ac5864b2-231c-45bd-8efa-594ea27cde2d"
           (reference "#PWR019") (unit 1)
@@
     (pin "8")
     (instances
-      (project "PCB-Controladora-Vuelo"
+      (project "PCB_Controladora_Vuelo_V2"
         (path "/ac5864b2-231c-45bd-8efa-594ea27cde2d"
           (reference "U1") (unit 1)
@@
         )
       )
-      (project "PCB-Controladora-Vuelo"
+      (project "PCB_Controladora_Vuelo_V2"
         (path "/ac5864b2-231c-45bd-8efa-594ea27cde2d"
           (reference "#PWR011") (unit 1)
@@
       (effects (font (size 1.016 1.016)) (justify left))
     )
-    (property "Footprint" "Capacitor_SMD:C_1206_3216Metric" (at 58.6232 60.452 0)
+    (property "Footprint" "EESTN5:C_0805" (at 58.6232 60.452 0)
       (effects (font (size 0.762 0.762)) hide)
     )
@@
         )
       )
-      (project "PCB-Controladora-Vuelo"
+      (project "PCB_Controladora_Vuelo_V2"
         (path "/ac5864b2-231c-45bd-8efa-594ea27cde2d"
           (reference "C7") (unit 1)
@@
         )
       )
-      (project "PCB-Controladora-Vuelo"
+      (project "PCB_Controladora_Vuelo_V2"
         (path "/ac5864b2-231c-45bd-8efa-594ea27cde2d"
           (reference "#PWR04") (unit 1)
@@
       (effects (font (size 1.27 1.27)) (justify left))
     )
-    (property "Footprint" "Capacitor_SMD:C_1206_3216Metric_Pad1.33x1.80mm_HandSolder" (at 50.7492 60.452 0)
+    (property "Footprint" "EESTN5:C_0805" (at 50.7492 60.452 0)
       (effects (font (size 1.27 1.27)) hide)
     )
@@
         )
       )
-      (project "PCB-Controladora-Vuelo"
+      (project "PCB_Controladora_Vuelo_V2"
         (path "/ac5864b2-231c-45bd-8efa-594ea27cde2d"
           (reference "C5") (unit 1)
@@
         )
       )
-      (project "PCB-Controladora-Vuelo"
+      (project "PCB_Controladora_Vuelo_V2"
         (path "/ac5864b2-231c-45bd-8efa-594ea27cde2d"
           (reference "#PWR010") (unit 1)
@@
     (pin "9")
     (instances
-      (project "PCB-Controladora-Vuelo"
+      (project "PCB_Controladora_Vuelo_V2"
         (path "/ac5864b2-231c-45bd-8efa-594ea27cde2d"
           (reference "U2") (unit 1)
@@
         )
       )
-      (project "PCB-Controladora-Vuelo"
+      (project "PCB_Controladora_Vuelo_V2"
         (path "/ac5864b2-231c-45bd-8efa-594ea27cde2d"
           (reference "#PWR015") (unit 1)
@@
         )
       )
-      (project "PCB-Controladora-Vuelo"
+      (project "PCB_Controladora_Vuelo_V2"
         (path "/ac5864b2-231c-45bd-8efa-594ea27cde2d"
           (reference "#PWR013") (unit 1)
@@
       (effects (font (size 1.016 1.016)) (justify left))
     )
-    (property "Footprint" "Capacitor_SMD:C_1206_3216Metric" (at 29.4132 60.452 0)
+    (property "Footprint" "EESTN5:C_0805" (at 29.4132 60.452 0)
       (effects (font (size 0.762 0.762)) hide)
     )
@@
         )
       )
-      (project "PCB-Controladora-Vuelo"
+      (project "PCB_Controladora_Vuelo_V2"
         (path "/ac5864b2-231c-45bd-8efa-594ea27cde2d"
           (reference "C3") (unit 1)
@@
     )
     (instances
-      (project "PCB-Controladora-Vuelo"
+      (project "PCB_Controladora_Vuelo_V2"
         (path "/ac5864b2-231c-45bd-8efa-594ea27cde2d"
           (reference "H4") (unit 1)
@@
         )
       )
-      (project "PCB-Controladora-Vuelo"
+      (project "PCB_Controladora_Vuelo_V2"
         (path "/ac5864b2-231c-45bd-8efa-594ea27cde2d"
           (reference "#PWR02") (unit 1)
@@
         )
       )
-      (project "PCB-Controladora-Vuelo"
+      (project "PCB_Controladora_Vuelo_V2"
         (path "/ac5864b2-231c-45bd-8efa-594ea27cde2d"
           (reference "#PWR012") (unit 1)
@@
     )
     (instances
-      (project "PCB-Controladora-Vuelo"
+      (project "PCB_Controladora_Vuelo_V2"
         (path "/ac5864b2-231c-45bd-8efa-594ea27cde2d"
           (reference "H3") (unit 1)
@@
         )
       )
-      (project "PCB-Controladora-Vuelo"
+      (project "PCB_Controladora_Vuelo_V2"
         (path "/ac5864b2-231c-45bd-8efa-594ea27cde2d"
           (reference "#PWR014") (unit 1)
@@
         )
       )
-      (project "PCB-Controladora-Vuelo"
+      (project "PCB_Controladora_Vuelo_V2"
         (path "/ac5864b2-231c-45bd-8efa-594ea27cde2d"
           (reference "U4") (unit 1)
@@
       (effects (font (size 1.27 1.27)) (justify left))
     )
-    (property "Footprint" "Capacitor_SMD:C_1206_3216Metric_Pad1.33x1.80mm_HandSolder" (at 23.0632 60.452 0)
+    (property "Footprint" "EESTN5:C_0805" (at 23.0632 60.452 0)
       (effects (font (size 1.27 1.27)) hide)
     )
@@
         )
       )
-      (project "PCB-Controladora-Vuelo"
+      (project "PCB_Controladora_Vuelo_V2"
         (path "/ac5864b2-231c-45bd-8efa-594ea27cde2d"
           (reference "C1") (unit 1)
@@
     (pin "2")
     (instances
-      (project "PCB-Controladora-Vuelo"
+      (project "PCB_Controladora_Vuelo_V2"
         (path "/ac5864b2-231c-45bd-8efa-594ea27cde2d"
           (reference "J1") (unit 1)
@@
         )
       )
-      (project "PCB-Controladora-Vuelo"
+      (project "PCB_Controladora_Vuelo_V2"
         (path "/ac5864b2-231c-45bd-8efa-594ea27cde2d"
           (reference "#PWR09") (unit 1)
@@
         )
       )
-      (project "PCB-Controladora-Vuelo"
+      (project "PCB_Controladora_Vuelo_V2"
         (path "/ac5864b2-231c-45bd-8efa-594ea27cde2d"
           (reference "U3") (unit 1)
